File: adc.kicad_pcb (KiCad board)
At the start: 2 copper layers, 8 parts, among them J1 Screw_Terminal_01x02, U1 Pico, U2 ADS8881CDGS, U3 LM4040DBZ-3

Commit message: update 06.02.2025
Parts:
- added C5: 100n, moja_biblioteka:cap_1206, F.Cu at (43.5, 75.7)
- added C6: 10u, moja_biblioteka:cap_1206, F.Cu at (43.5, 79.5)
- added C7: 100n, moja_biblioteka:cap_1206, F.Cu at (43.5, 83.2)
- added R1: 100, moja_biblioteka:res_1206, F.Cu at (54.2, 75.2)
- added U4: OPA320AIDBVR, OPA320:DBV5, F.Cu at (51.5, 78.3)
- C1: value 100n -> 10u
- C3, C4: value 100n -> 1u
- moved J1 95.1 mm to (42.0, 48.0), turned to -90 degrees
- moved C2 67.7 mm to (53.5, 61.6)
- moved U3 66.6 mm to (57.5, 52.5)
- moved C4 58.8 mm to (63.0, 70.7)
- moved C3 55.8 mm to (64.0, 43.6)
- moved U2 55.7 mm to (70.5, 47.0)
- moved C1 55.0 mm to (66.0, 55.6)
Connections:
- J1 pad 1: DIODE_IN -> Net-(J1-Pin_1)

Commit message: Add files via upload
Parts:
- added C1: 1u, moja_biblioteka:cap_1206, F.Cu at (7.75, 2.55)
- added C10: 100n, moja_biblioteka:cap_1206, F.Cu at (14.2, 10.2)
- added C11: 10u, moja_biblioteka:cap_1206, F.Cu at (14.2, 13.9)
- added C12: 10n, moja_biblioteka:cap_1206, F.Cu at (14.2, 17.8)
- added C13: 10n, moja_biblioteka:cap_1206, F.Cu at (14.2, 21.6)
- added C14: 10u, moja_biblioteka:cap_1206, F.Cu at (20.8, 2.55)
- added C15: 10n, moja_biblioteka:cap_1206, F.Cu at (20.8, 6.35)
- added C16: 10n, moja_biblioteka:cap_1206, F.Cu at (20.8, 10.2)
- added C17: 10u, moja_biblioteka:cap_1206, F.Cu at (20.8, 13.9)
- added C2: 1u, moja_biblioteka:cap_1206, F.Cu at (7.75, 6.35)
- added C3: 1u, moja_biblioteka:cap_1206, F.Cu at (7.75, 10.2)
- added C4: 10u, moja_biblioteka:cap_1206, F.Cu at (7.75, 13.9)
- added C5: 10u, moja_biblioteka:cap_1206, F.Cu at (7.75, 17.8)
- added C6: 1u, moja_biblioteka:cap_1206, F.Cu at (7.75, 21.6)
- added C8: 10n, moja_biblioteka:cap_1206, F.Cu at (14.2, 2.55)
- added C9: 100n, moja_biblioteka:cap_1206, F.Cu at (14.2, 6.35)
- added J2: Screw_Terminal_01x02, moja_biblioteka:screw_conector, F.Cu at (9.85, 26.9)
- added R10: 1k, moja_biblioteka:res_1206, F.Cu at (5.00, 28.9)
- added R11: 1k, moja_biblioteka:res_1206, F.Cu at (5.00, 32.2)
- added R12: 4.7k, moja_biblioteka:res_1206, F.Cu at (5.00, 35.6)
- added R13: 1k, moja_biblioteka:res_1206, F.Cu at (5.00, 39.0)
- added R14: 100, moja_biblioteka:res_1206, F.Cu at (-2.00, 35.6)
- added R15: 10k, moja_biblioteka:res_1206, F.Cu at (-2.00, 39.0)
- added R2: 1k, moja_biblioteka:res_1206, F.Cu at (5.00, 2.10)
- added R3: 0.2, moja_biblioteka:res_1206, F.Cu at (5.00, 5.45)
- added R4: 1k, moja_biblioteka:res_1206, F.Cu at (5.00, 8.80)
- added R5: 20k, moja_biblioteka:res_1206, F.Cu at (5.00, 12.2)
- added R6: 10, moja_biblioteka:res_1206, F.Cu at (5.00, 15.5)
- added R7: 10, moja_biblioteka:res_1206, F.Cu at (5.00, 18.9)
- added R8: 1k, moja_biblioteka:res_1206, F.Cu at (5.00, 22.2)
- added R9: 1k, moja_biblioteka:res_1206, F.Cu at (5.00, 25.6)
- added U3: LM4040DBZ-3, Package_TO_SOT_SMD:SOT-23, F.Cu at (20.5, 33.2)
- added U5: THS4521ID, Package_SO:SOIC-8_3.9x4.9mm_P1.27mm, F.Cu at (30.2, 2.85)
- added U6: OPA333xxD, Package_SO:SOIC-8_3.9x4.9mm_P1.27mm, F.Cu at (30.2, 9.44)
- added U7: REF5045AD, Package_SO:SOIC-8_3.9x4.9mm_P1.27mm, F.Cu at (30.2, 16.0)
- added U8: THS4281, moja_biblioteka:THS4281, F.Cu at (19.6, 23.7)
- added U9: TPS7A49, moja_biblioteka:TPS7A49, F.Cu at (19.6, 27.9)
- C7: value 100n -> 33u
Connections:
- C7 pad 1: DIODE_IN -> Net-(U4-IN-)
- C7 pad 2: GND -> DIODE_IN
- R1 pad 1: Net-(U4-IN-) -> DIODE_IN
- R1 pad 2: DIODE_IN -> GND
- U1 pad 7: trig -> unconnected-(U1-GPIO5-Pad7)
- U2 pad 1: 3.3V -> V_REF
- U2 pad 10: 3.3V -> +3
- U2 pad 2: 3.3V -> +3
- U2 pad 3: DIODE_IN -> Net-(U2-AINP)
- U2 pad 4: GND -> Net-(U2-AINM)
- U4 pad 5: 3.3V -> +3

Commit message: Add files via upload
Parts:
- added C4: 33u, moja_biblioteka:cap_1206, F.Cu at (118.2, 47.1)
- added D1: SMAJ12A, Diode_SMD:D_SMA, F.Cu at (121.1, 41.8)
- added D2: LED, moja_biblioteka:LED_SMD, F.Cu at (118.0, 48.9)
- added R1: 100, moja_biblioteka:res_1206, F.Cu at (115.5, 42.1)
- added R16: 400, moja_biblioteka:res_1206, F.Cu at (115.5, 45.4)
- added R17: 470, moja_biblioteka:res_1206, F.Cu at (115.5, 48.8)
- added R18: 10k, moja_biblioteka:res_1206, F.Cu at (115.5, 52.1)
- added R19: 100, moja_biblioteka:res_1206, F.Cu at (115.5, 55.5)
- C12, C13: value 10n -> 1u
- moved R10 125.2 mm to (115.0, 88.8)
- moved R11 125.2 mm to (115.0, 92.1)
- moved R12 125.2 mm to (115.0, 95.5)
- moved R13 125.2 mm to (115.0, 98.8)
- moved R14 125.2 mm to (108.0, 95.5)
- moved R15 125.2 mm to (108.0, 98.8)
- moved R2 125.2 mm to (115.0, 62.0)
- moved R3 125.2 mm to (115.0, 65.3)
- moved R4 125.2 mm to (115.0, 68.7)
- moved R5 125.2 mm to (115.0, 72.0)
- moved R6 125.2 mm to (115.0, 75.3)
- moved R7 125.2 mm to (115.0, 78.7)
- moved R8 125.2 mm to (115.0, 82.0)
- moved R9 125.2 mm to (115.0, 85.4)
- moved C1 55.1 mm to (42.5, 45.2)
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Connections:
- C16 pad 1: +3 -> +5
- C17 pad 1: +3 -> +5
- R11 pad 2: DIODE_IN -> DIODE_SIGNAL
- R12 pad 1: +3 -> +5
- R14 pad 1: +3 -> +5
- U4 pad 1: Net-(U4-IN-) -> DIODE_SIGNAL
- U4 pad 3: Net-(J1-Pin_1) -> Net-(U4-+)
- U4 pad 4: Net-(U4-IN-) -> Net-(U4--)
- U4 pad 5: +3 -> +5
- U5 pad 3: +3 -> +5
- U5 pad 7: +3 -> +5
- U6 pad 7: +3 -> +5
- U7 pad 2: +3 -> +5
- U8 pad 5: +3 -> +5
- U9 pad 1: +3 -> +5
Other:
- board outline added: 92 x 69.5 mm
