File: adc.kicad_sch (KiCad schematic)
At the start: 8 parts, among them J1 Screw_Terminal_01x02, U1 Pico, U2 ADS8881CDGS, U3 LM4040DBZ-3

Commit message: update 06.02.2025
Parts:
- added C10, C9: 100n, moja_biblioteka:cap_1206, symbol moja_biblioteka:cap_1206
- added C11, C14, C17, C5: 10u, moja_biblioteka:cap_1206, symbol moja_biblioteka:cap_1206
- added C12, C13, C15, C16, C8: 10n, moja_biblioteka:cap_1206, symbol moja_biblioteka:cap_1206
- added C6: 1u, moja_biblioteka:cap_1206, symbol moja_biblioteka:cap_1206
- added C7: 33u, moja_biblioteka:cap_1206, symbol moja_biblioteka:cap_1206
- added J2: Screw_Terminal_01x02, moja_biblioteka:screw_conector, symbol moja_biblioteka:Screw_Terminal_01x02
- added R1: 100, moja_biblioteka:res_1206, symbol moja_biblioteka:res_1206
- added R10, R11, R2, R4, R8, R9: 1k, moja_biblioteka:res_1206, symbol moja_biblioteka:res_1206
- added R12: 33k, moja_biblioteka:res_1206, symbol moja_biblioteka:res_1206
- added R13: 10k, moja_biblioteka:res_1206, symbol moja_biblioteka:res_1206
- added R3: 0.2, moja_biblioteka:res_1206, symbol moja_biblioteka:res_1206
- added R5: 20k, moja_biblioteka:res_1206, symbol moja_biblioteka:res_1206
- added R6, R7: 10, moja_biblioteka:res_1206, symbol moja_biblioteka:res_1206
- added U4: OPA320AIDBVR, OPA320:DBV5, symbol OPA320:OPA320AIDBVR
- added U5: THS4521ID, Package_SO:SOIC-8_3.9x4.9mm_P1.27mm, symbol Amplifier_Difference:THS4521ID
- added U6: OPA333xxD, Package_SO:SOIC-8_3.9x4.9mm_P1.27mm, symbol Amplifier_Operational:OPA333xxD
- added U7: REF5045AD, Package_SO:SOIC-8_3.9x4.9mm_P1.27mm, symbol Reference_Voltage:REF5045AD
- added U8: THS4281, moja_biblioteka:THS4281, symbol moja_biblioteka:THS4281
- added U9: TPS7A49, moja_biblioteka:THS4281, symbol moja_biblioteka:TPS7A49
- C1, C2, C3: value 100n -> 1u
- C4: value 100n -> 10u
Connections:
- net 3.3V: no longer C1.1, C2.1, C3.1, C4.1, U2.1 (REF), U2.10 (DVDD), U2.2 (AVDD), U3.1 (K)
- net DIODE_IN: now also C7.2, R1.1, R11.2; no longer J1.1 (Pin_1), U2.3 (AINP)
- net GND: now also C10.2, C11.2, C12.2, C13.2, C14.2, C15.2, C17.2, C5.2, C6.2, C9.2, J2.2 (Pin_2), R1.2, R13.2, R9.1, U4.2 (V-), U5.6 (V_{S-}), U6.4 (V-), U7.4 (GND), U8.2 (V-), U9.4 (GND); no longer C1.2, U2.4 (AINN)
- net trig: no longer names the net of U1.7 (GPIO5)
- new net: C3.1, U7.5 (Trim/NR)
- new net: R7.2, R8.1, U5.4
- new net: R8.2, R9.2, U5.1 (-)
- new net: C8.2, R7.1, U2.4 (AINM)
- new net: C15.1, U9.6 (NE/SS)
- new net: C16.2, R12.2, R13.1, U9.2 (FB)
- new net: C14.1, J2.1 (Pin_1), U9.5 (EN), U9.8 (IN)
- new net: C8.1, R6.1, U2.3 (AINP)
- new net: R10.1, R6.2, U5.5
- new net: C6.1, R2.2, U6.3 (+)
- new net: C7.1, U4.1 (OUT), U4.4 (IN-)
- new net: J1.1 (Pin_1), U4.3 (IN+)
- new net: C1.2, R5.1, U6.2 (-)
- new net: C1.1, R4.1, U6.6
- new net: R10.2, R11.1, U5.8 (+)
- new net: C5.1, R3.2
- new net: R2.1, U7.6 (Vout)
- new net: C2.1, R4.2, U8.1 (+)
- new net +3: C10.1, C11.1, C12.1, C13.1, C16.1, C17.1, C4.1, C9.1, R12.1, U2.10 (DVDD), U2.2 (AVDD), U3.1 (K), U4.5 (V+), U5.3 (V_{S+}), U5.7 (~{PD}), U6.7 (V+), U7.2 (Vin), U8.5 (V+), U9.1 (OUT)
- new net V_REF: R3.1, R5.2, U2.1 (REF), U5.2 (V_{OCM}), U8.1 (+), U8.3 (-)
- no-connect marks 0 -> 1
Other:
- note added: "5V = 1,188V * (1 + R1/R2) R1/R2 = 5/1,188 - 1 = 3,21 33kΩ / 10kΩ = 3,3"
- note added: "ADC"
- note added: "KONDENSATORY"
- note added: "LDO V_IN = 12V, V_OUT = 5V"
- note added: "ODSPRZEGAJACE ADS8881"
- note added: "RPI PICO"
- note added: "STABILIZATOR NAPIECIA 3V"
- note added: "SYGNAL WEJSCIOWY"
- note added: "V_REF 5V"
- note added: "V_REF = 1.188V (napięcie referencyjne układu TPS7A4901), V_OUT = 5V (założone napięcie wyjściowe),"
- note added: "t_ss [ms] = 1,4 * C_NR/SS [nF] t_ss = 1,4 * 10nF = 14 ms"
- moved on the sheet: J1, U1, U2

Commit message: Add files via upload
Parts:
- added R14: 100, moja_biblioteka:res_1206, symbol moja_biblioteka:res_1206
- added R15: 10k, moja_biblioteka:res_1206, symbol moja_biblioteka:res_1206
- R12: value 33k -> 4.7k
- R13: value 10k -> 1k
- U9: footprint moja_biblioteka:THS4281 -> moja_biblioteka:TPS7A49
Connections:
- net +3: now also R14.1
- net V_REF: now also U8.4 (-); no longer U8.3 (-)
- net at C16.2, R12.2, R13.1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: now also R15.2
- net at C2.1, R4.2: now also U8.3 (+); no longer U8.1 (+)
- new net: R14.2, R15.1
Other:
- note added: "5V = 1,188V * (1 + R1/R2) R1/R2 = 5/1,188 - 1 = 3,21 4,7kΩ || 10,1kΩ = 3,21kΩ 3,21kΩ / 1k = 3,21"
- note added: "ODSPRZĘGAJĄCE ADS8881"
- note added: "STABILIZATOR NAPIĘCIA 3V"
- note added: "SYGNAŁ WEJŚCIOWY"
- note removed: "5V = 1,188V * (1 + R1/R2) R1/R2 = 5/1,188 - 1 = 3,21 33kΩ / 10kΩ = 3,3"
- note removed: "ODSPRZEGAJACE ADS8881"
- note removed: "STABILIZATOR NAPIECIA 3V"
- note removed: "SYGNAL WEJSCIOWY"
- company: (none) -> Politechnika Wrocławska
- title: (none) -> mini-project ADC
- moved on the sheet: C16, R12, R13

Commit message: Add files via upload
Parts:
- C12, C13: value 10n -> 1u
Other:
- note added: "dodać diody TVS i/lub bezpieczniki"
- note added: "filtr górnoprzepustowy f_g = 48 Hz"
Changed lines of the file:
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@@
 	(rectangle
 		(start 12.7 67.31)
-		(end 95.25 99.06)
+		(end 96.52 104.14)
 		(stroke
 			(width 0)
@@
 	(text "SYGNAŁ WEJŚCIOWY"
 		(exclude_from_sim no)
-		(at 76.2 97.79 0)
+		(at 76.454 99.568 0)
 		(effects
 			(font
@@
 		)
 	)
+	(text "dodać diody TVS \ni/lub bezpieczniki"
+		(exclude_from_sim no)
+		(at 35.56 16.256 0)
+		(effects
+			(font
+				(size 1.27 1.27)
+			)
+		)
+	)
 	(text "V_REF = 1.188V (napięcie referencyjne układu TPS7A4901),\nV_OUT = 5V (założone napięcie wyjściowe),"
 		(exclude_from_sim no)
@@
 		)
 	)
+	(text "filtr górnoprzepustowy f_g = 48 Hz"
+		(exclude_from_sim no)
+		(at 78.232 102.362 0)
+		(effects
+			(font
+				(size 1.27 1.27)
+			)
+		)
+	)
 	(text "KONDENSATORY"
 		(exclude_from_sim no)
@@
 	(text "t_ss [ms] = 1,4 * C_NR/SS [nF]\nt_ss = 1,4 * 10nF = 14 ms"
 		(exclude_from_sim no)
-		(at 78.232 50.546 0)
+		(at 78.486 53.086 0)
 		(effects
 			(font
@@
 			)
 		)
-		(property "Value" "10n"
+		(property "Value" "1u"
 			(at 283.972 25.146 90)
 			(effects
@@
 			)
 		)
-		(property "Value" "10n"
+		(property "Value" "1u"
 			(at 273.812 25.146 90)
 			(effects

Commit message: Add files via upload
Parts:
- removed C11: 10u, moja_biblioteka:cap_1206, symbol moja_biblioteka:cap_1206
- removed C7: 33u, moja_biblioteka:cap_1206, symbol moja_biblioteka:cap_1206
- removed C9: 100n, moja_biblioteka:cap_1206, symbol moja_biblioteka:cap_1206
- added D1: SMAJ12A, Diode_SMD:D_SMA, symbol Diode:SMAJ12A
- added D2: LED, moja_biblioteka:LED_SMD, symbol moja_biblioteka:LED_SMD
- added R16: 400, moja_biblioteka:res_1206, symbol moja_biblioteka:res_1206
- added R17: 470, moja_biblioteka:res_1206, symbol moja_biblioteka:res_1206
- added R18: 10k, moja_biblioteka:res_1206, symbol moja_biblioteka:res_1206
- added R19: 100, moja_biblioteka:res_1206, symbol moja_biblioteka:res_1206
- C4: value 10u -> 33u
Connections:
- net +3: now also R16.2; no longer C16.1, C17.1, C4.1, R12.1, R14.1, U4.5 (V+), U5.3 (V_{S+}), U5.7 (~{PD}), U6.7 (V+), U7.2 (Vin), U8.5 (V+), U9.1 (OUT)
- net GND: now also D1.2 (A2), R17.2, R19.2; no longer C4.2
- net at C14.1, J2.1 (Pin_1), U9.5 (EN)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: now also D1.1 (A1)
- net at U4.4 (-): now also R18.2, R19.1; no longer U4.1 (OUT)
- net at U4.3 (+): now also C4.2, R1.1; no longer J1.1 (Pin_1)
- net DIODE_IN renamed DIODE_SIGNAL
- net DIODE_SIGNAL: now also U4.1, R18.1; no longer R1.1
- new net: D2.1 (K), R17.1
- new net: C4.1, J1.1 (Pin_1)
- new net +5: C16.1, C17.1, D2.2 (A), R12.1, R14.1, R16.1, U4.5 (V+), U5.3 (V_{S+}), U5.7 (~{PD}), U6.7 (V+), U7.2 (Vin), U8.5 (V+), U9.1 (OUT)
- no-connect marks 1 -> 37
Other:
- note added: "4,5V REFERANCE VOLTAGE FOR ADC"
- note added: "ANALOG TO DIGITAL CONVERTER"
- note added: "DECOUPLONG CAPACITORS FOR ADC"
- note added: "GAIN = R18/R19 + 1 GAIN = 10k / 100 + 1 = 101"
- note added: "HIGHPASS FILTER f_g = 48 Hz"
- note added: "OUTPUT SIGNAL FROM DIODE"
- note added: "REFERANCE VOLTAGE 3V FOR ADC"
- note added: "V_REF = 1.188V (voltage referance of TPS7A4901), V_OUT = 5V (output voltage),"
- note removed: "ADC"
- note removed: "KONDENSATORY"
- note removed: "ODSPRZĘGAJĄCE ADS8881"
- note removed: "STABILIZATOR NAPIĘCIA 3V"
- note removed: "SYGNAŁ WEJŚCIOWY"
- note removed: "V_REF 5V"
- note removed: "V_REF = 1.188V (napięcie referencyjne układu TPS7A4901), V_OUT = 5V (założone napięcie wyjściowe),"
- note removed: "dodać diody TVS i/lub bezpieczniki"
- note removed: "filtr górnoprzepustowy f_g = 48 Hz"
- moved on the sheet: C1, C10, C12, C13, C14, C15, C16, C17, C2, C3, C5, C6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
